File: eagle/4th_MFB_LPF/4th_MFB_LPF.brd (EAGLE design)
At the start: 30.1 x 40.6 mm, 16 parts, among them IC1 NJM2068

Commit message: 回路図修正
Connections:
- net V+: now also C6.1, IC1.8, JP1.2; no longer C5.1, IC1.4, JP1.3
- net V-: now also C5.1, IC1.4, JP1.3; no longer C6.1, IC1.8, JP1.2
Routing:
- net V-: track 16.3 -> 8.67 mm
- net V+: track 8.67 -> 16.3 mm
Other:
- board size 30.1 x 40.6 mm -> 31.4 x 40.6 mm
Changed lines of the file:
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@@
 <board>
 <plain>
-<wire x1="0" y1="0" x2="30.15" y2="0" width="0" layer="20"/>
-<wire x1="30.15" y1="0" x2="30.15" y2="40.63" width="0" layer="20"/>
-<wire x1="30.15" y1="40.63" x2="0" y2="40.63" width="0" layer="20"/>
+<wire x1="0" y1="0" x2="31.42" y2="0" width="0" layer="20"/>
+<wire x1="31.42" y1="0" x2="31.42" y2="40.63" width="0" layer="20"/>
+<wire x1="31.42" y1="40.63" x2="0" y2="40.63" width="0" layer="20"/>
 <wire x1="0" y1="40.63" x2="0" y2="0" width="0" layer="20"/>
 <wire x1="2.54" y1="2.54" x2="15.24" y2="2.54" width="0" layer="100"/>
@@
 <signals>
 <signal name="V-">
+<contactref element="IC1" pad="4"/>
+<contactref element="C5" pad="1"/>
+<contactref element="JP1" pad="3"/>
+<wire x1="22.86" y1="15.24" x2="25.4" y2="15.24" width="0.4064" layer="16"/>
+<wire x1="25.4" y1="15.24" x2="27.94" y2="17.78" width="0.4064" layer="16"/>
+<wire x1="22.86" y1="15.24" x2="22.86" y2="12.7" width="0.4064" layer="16"/>
+</signal>
+<signal name="V+">
+<contactref element="C6" pad="1"/>
 <contactref element="IC1" pad="8"/>
-<contactref element="C6" pad="1"/>
 <contactref element="JP1" pad="2"/>
 <wire x1="12.7" y1="22.86" x2="15.24" y2="22.86" width="0.4064" layer="16"/>
@@
 <wire x1="26.67" y1="21.59" x2="27.94" y2="20.32" width="0.4064" layer="1"/>
 </signal>
-<signal name="V+">
-<contactref element="IC1" pad="4"/>
-<contactref element="C5" pad="1"/>
-<contactref element="JP1" pad="3"/>
-<wire x1="22.86" y1="15.24" x2="22.86" y2="12.7" width="0.4064" layer="16"/>
-<wire x1="22.86" y1="15.24" x2="25.4" y2="15.24" width="0.4064" layer="16"/>
-<wire x1="25.4" y1="15.24" x2="27.94" y2="17.78" width="0.4064" layer="16"/>
-</signal>
 <signal name="GND">
